File: KiCAD/Drone_Flight_Controller/Battery Monitoring.kicad_sch (KiCad schematic)
At the start: 7 parts, among them U205 AS358

Commit message: Fix errors
Connections:
- net -BATT renamed GND
Changed lines of the file:
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@@
 	(title_block
 		(title "Battery Monitoring")
-		(date "2025-09-19")
+		(date "2025-09-21")
 		(rev "V2")
 		(company "HTL Steyr")
@@
 	)
 	(symbol
+		(lib_id "power:GND")
+		(at 105.41 30.48 0)
+		(unit 1)
+		(exclude_from_sim no)
+		(in_bom yes)
+		(on_board yes)
+		(dnp no)
+		(fields_autoplaced yes)
+		(property "Reference" "#PWR02"
+			(at 105.41 36.83 0)
+			(effects
+				(font
+					(size 1.27 1.27)
+				)
+				(hide yes)
+			)
+		)
+		(property "Value" "GND"
+			(at 105.41 35.56 0)
+			(effects
+				(font
+					(size 1.27 1.27)
+				)
+			)
+		)
+		(property "Footprint" ""
+			(at 105.41 30.48 0)
+			(effects
+				(font
+					(size 1.27 1.27)
+				)
+				(hide yes)
+			)
+		)
+		(property "Datasheet" ""
+			(at 105.41 30.48 0)
+			(effects
+				(font
+					(size 1.27 1.27)
+				)
+				(hide yes)
+			)
+		)
+		(property "Description" "Power symbol creates a global label with name \"GND\" , ground"
+			(at 105.41 30.48 0)
+			(effects
+				(font
+					(size 1.27 1.27)
+				)
+				(hide yes)
+			)
+		)
+		(pin "1"
+		)
+		(instances
+			(project ""
+				(path "/05daaa24-e506-4b9a-9564-8bf799413ca8/8aeacdae-c3f2-480a-a34d-37642627b117"
+					(reference "#PWR02")
+					(unit 1)
+				)
+			)
+		)
+	)
+	(symbol
 		(lib_id "Device:R")
 		(at 78.74 44.45 90)
@@
 					(unit 1)
 				)
-			)
-		)
-	)
-	(symbol
-		(lib_id "power:-BATT")
-		(at 105.41 30.48 180)
-		(unit 1)
-		(exclude_from_sim no)
-		(in_bom yes)
-		(on_board yes)
-		(dnp no)
-		(fields_autoplaced yes)
-		(property "Reference" "#PWR0501"
-			(at 105.41 26.67 0)
-			(effects
-				(font
-					(size 1.27 1.27)
-				)
-				(hide yes)
-			)
-		)
-		(property "Value" "-BATT"
-			(at 105.41 35.56 0)
-			(effects
-				(font
-					(size 1.27 1.27)
-				)
-			)
-		)
-		(property "Footprint" ""
-			(at 105.41 30.48 0)
-			(effects
-				(font
-					(size 1.27 1.27)
-				)
-				(hide yes)
-			)
-		)
-		(property "Datasheet" ""
-			(at 105.41 30.48 0)
-			(effects
-				(font
-					(size 1.27 1.27)
-				)
-				(hide yes)
-			)
-		)
-		(property "Description" "Power symbol creates a global label with name \"-BATT\""
-			(at 105.41 30.48 0)
-			(effects
-				(font
-					(size 1.27 1.27)
-				)
-				(hide yes)
-			)
-		)
-		(pin "1"
-		)
-		(instances
-			(project ""
-				(path "/05daaa24-e506-4b9a-9564-8bf799413ca8/8aeacdae-c3f2-480a-a34d-37642627b117"
-					(reference "#PWR0501")
-					(unit 1)
-				)

Commit message: Cleanup & Re-annotate
Parts:
- renumbered R502 to R601, R503 to R602, R504 to R603, R505 to R604, R501 to R605, R506 to R606, U205 to U301
Changed lines of the file:
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@@
 		(on_board yes)
 		(dnp no)
-		(property "Reference" "R505"
+		(property "Reference" "R604"
 			(at 90.17 53.34 90)
 			(effects
@@
 			(project "Drone_Flight_Controller"
 				(path "/05daaa24-e506-4b9a-9564-8bf799413ca8/8aeacdae-c3f2-480a-a34d-37642627b117"
-					(reference "R505")
+					(reference "R604")
 					(unit 1)
 				)
@@
 		(on_board yes)
 		(dnp no)
-		(property "Reference" "R506"
+		(property "Reference" "R606"
 			(at 100.33 53.34 90)
 			(effects
@@
 			(project "Drone_Flight_Controller"
 				(path "/05daaa24-e506-4b9a-9564-8bf799413ca8/8aeacdae-c3f2-480a-a34d-37642627b117"
-					(reference "R506")
+					(reference "R606")
 					(unit 1)
 				)
@@
 		(dnp no)
 		(fields_autoplaced yes)
-		(property "Reference" "R501"
+		(property "Reference" "R605"
 			(at 95.25 21.59 90)
 			(effects
@@
 			(project ""
 				(path "/05daaa24-e506-4b9a-9564-8bf799413ca8/8aeacdae-c3f2-480a-a34d-37642627b117"
-					(reference "R501")
+					(reference "R605")
 					(unit 1)
 				)
@@
 		(dnp no)
 		(fields_autoplaced yes)
-		(property "Reference" "U205"
+		(property "Reference" "U301"
 			(at 118.11 34.29 0)
 			(effects
@@
 			(project "Drone_Flight_Controller"
 				(path "/05daaa24-e506-4b9a-9564-8bf799413ca8/8aeacdae-c3f2-480a-a34d-37642627b117"
-					(reference "U205")
+					(reference "U301")
 					(unit 2)
 				)
@@
 		(dnp no)
 		(fields_autoplaced yes)
-		(property "Reference" "U205"
+		(property "Reference" "U301"
 			(at 95.25 31.75 0)
 			(effects
@@
 			(project "Drone_Flight_Controller"
 				(path "/05daaa24-e506-4b9a-9564-8bf799413ca8/8aeacdae-c3f2-480a-a34d-37642627b117"
-					(reference "U205")
+					(reference "U301")
 					(unit 1)
 				)
@@
 		(dnp no)
 		(fields_autoplaced yes)
-		(property "Reference" "#PWR02"
+		(property "Reference" "#PWR0602"
 			(at 105.41 36.83 0)
 			(effects
@@
 			(project ""
 				(path "/05daaa24-e506-4b9a-9564-8bf799413ca8/8aeacdae-c3f2-480a-a34d-37642627b117"
-					(reference "#PWR02")
+					(reference "#PWR0602")
 					(unit 1)
 				)
@@
 		(on_board yes)
 		(dnp no)
-		(property "Reference" "R504"
+		(property "Reference" "R603"
 			(at 78.74 47.244 90)
 			(effects
@@
 			(project "Drone_Flight_Controller"
 				(path "/05daaa24-e506-4b9a-9564-8bf799413ca8/8aeacdae-c3f2-480a-a34d-37642627b117"
-					(reference "R504")
+					(reference "R603")
 					(unit 1)
 				)
@@
 		(dnp no)
 		(fields_autoplaced yes)
-		(property "Reference" "#+3V0101"
+		(property "Reference" "#+3V0601"
 			(at 40.64 36.83 0)
 			(effects
@@
 			(project ""
 				(path "/05daaa24-e506-4b9a-9564-8bf799413ca8/8aeacdae-c3f2-480a-a34d-37642627b117"
-					(reference "#+3V0101")
+					(reference "#+3V0601")
 					(unit 1)
 				)
@@
 		(dnp no)
 		(fields_autoplaced yes)
-		(property "Reference" "#PWR0503"
+		(property "Reference" "#PWR0601"
 			(at 50.8 36.83 0)
 			(effects
@@
 			(project ""
 				(path "/05daaa24-e506-4b9a-9564-8bf799413ca8/8aeacdae-c3f2-480a-a34d-37642627b117"
-					(reference "#PWR0503")
+					(reference "#PWR0601")
 					(unit 1)
 				)
@@
 		(dnp no)
 		(fields_autoplaced yes)
-		(property "Reference" "R502"
+		(property "Reference" "R601"
 			(at 68.58 33.02 90)
 			(effects
@@
 			(project ""
 				(path "/05daaa24-e506-4b9a-9564-8bf799413ca8/8aeacdae-c3f2-480a-a34d-37642627b117"
-					(reference "R502")
+					(reference "R601")
 					(unit 1)
 				)
@@
 		(dnp no)
 		(fields_autoplaced yes)
-		(property "Reference" "R503"
+		(property "Reference" "R602"
 			(at 78.74 33.02 90)
 			(effects
@@
 			(project "Drone_Flight_Controller"
 				(path "/05daaa24-e506-4b9a-9564-8bf799413ca8/8aeacdae-c3f2-480a-a34d-37642627b117"
-					(reference "R503")
-					(unit 1)
-				)
+					(reference "R602")
+					(unit 1)
+				)
