File: KiCAD/Drone_Flight_Controller/Buzzer.kicad_sch (KiCad schematic)
At the start: 4 parts, among them Q401 2N2222A

Commit message: Cleanup & Re-annotate
Parts:
- renumbered BZ401 to BZ501, Q401 to Q501, R402 to R501, R401 to R502
Changed lines of the file:
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@@
 		(dnp no)
 		(fields_autoplaced yes)
-		(property "Reference" "R402"
+		(property "Reference" "R501"
 			(at 106.68 99.06 90)
 			(effects
@@
 			(project ""
 				(path "/05daaa24-e506-4b9a-9564-8bf799413ca8/be7f0ff9-fd1d-432b-97a6-9126ad5ddcf4"
-					(reference "R402")
+					(reference "R501")
 					(unit 1)
 				)
@@
 		(dnp no)
 		(fields_autoplaced yes)
-		(property "Reference" "BZ401"
+		(property "Reference" "BZ501"
 			(at 135.89 90.1699 0)
 			(effects
@@
 			(project "Drone_Flight_Controller"
 				(path "/05daaa24-e506-4b9a-9564-8bf799413ca8/be7f0ff9-fd1d-432b-97a6-9126ad5ddcf4"
-					(reference "BZ401")
+					(reference "BZ501")
 					(unit 1)
 				)
@@
 		(dnp no)
 		(fields_autoplaced yes)
-		(property "Reference" "#+3V3"
+		(property "Reference" "#+3V0501"
 			(at 120.65 86.36 0)
 			(effects
@@
 			(project ""
 				(path "/05daaa24-e506-4b9a-9564-8bf799413ca8/be7f0ff9-fd1d-432b-97a6-9126ad5ddcf4"
-					(reference "#+3V3")
+					(reference "#+3V0501")
 					(unit 1)
 				)
@@
 		(dnp no)
 		(fields_autoplaced yes)
-		(property "Reference" "R401"
+		(property "Reference" "R502"
 			(at 123.19 90.1699 0)
 			(effects
@@
 			(project ""
 				(path "/05daaa24-e506-4b9a-9564-8bf799413ca8/be7f0ff9-fd1d-432b-97a6-9126ad5ddcf4"
-					(reference "R401")
+					(reference "R502")
 					(unit 1)
 				)
@@
 		(dnp no)
 		(fields_autoplaced yes)
-		(property "Reference" "Q401"
+		(property "Reference" "Q501"
 			(at 123.19 104.1399 0)
 			(effects
@@
 			(project ""
 				(path "/05daaa24-e506-4b9a-9564-8bf799413ca8/be7f0ff9-fd1d-432b-97a6-9126ad5ddcf4"
-					(reference "Q401")
+					(reference "Q501")
 					(unit 1)
 				)
@@
 		(dnp no)
 		(fields_autoplaced yes)
-		(property "Reference" "#PWR0402"
+		(property "Reference" "#PWR0501"
 			(at 120.65 119.38 0)
 			(effects
@@
 			(project ""
 				(path "/05daaa24-e506-4b9a-9564-8bf799413ca8/be7f0ff9-fd1d-432b-97a6-9126ad5ddcf4"
-					(reference "#PWR0402")
-					(unit 1)
-				)
+					(reference "#PWR0501")
+					(unit 1)
+				)
