File: KiCAD/Drone_Flight_Controller/uC and sensors.kicad_sch (KiCad schematic)
At the start: 11 parts, among them SW301 SW_Push, U301 DPS368, U302 BNO055, U303 ESP32-WROOM-32

Commit message: Cleanup & Re-annotate
Parts:
- C402: renamed from C302; value 120nF -> 120n
- C403: renamed from C301; value 1µF -> 1µ
- renumbered C304 to C401, C303 to C404, R301 to R401, R303 to R402, R302 to R403, SW301 to SW401, U301 to U401, U302 to U402, U303 to U403
Changed lines of the file:
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@@
 		(on_board yes)
 		(dnp no)
-		(property "Reference" "U303"
+		(property "Reference" "U403"
 			(at 179.578 103.632 90)
 			(effects
@@
 			(project "Drone_Flight_Controller"
 				(path "/05daaa24-e506-4b9a-9564-8bf799413ca8/be1bc5c9-9814-4f01-a307-b935c6145e5a"
-					(reference "U303")
+					(reference "U403")
 					(unit 1)
 				)
@@
 		(dnp no)
 		(fields_autoplaced yes)
-		(property "Reference" "#PWR0307"
+		(property "Reference" "#PWR0404"
 			(at 95.25 118.11 0)
 			(effects
@@
 			(project "Drone_Flight_Controller"
 				(path "/05daaa24-e506-4b9a-9564-8bf799413ca8/be1bc5c9-9814-4f01-a307-b935c6145e5a"
-					(reference "#PWR0307")
+					(reference "#PWR0404")
 					(unit 1)
 				)
@@
 		(dnp no)
 		(fields_autoplaced yes)
-		(property "Reference" "#PWR0302"
+		(property "Reference" "#PWR0403"
 			(at 95.25 69.85 0)
 			(effects
@@
 			(project ""
 				(path "/05daaa24-e506-4b9a-9564-8bf799413ca8/be1bc5c9-9814-4f01-a307-b935c6145e5a"
-					(reference "#PWR0302")
+					(reference "#PWR0403")
 					(unit 1)
 				)
@@
 		(on_board yes)
 		(dnp no)
-		(property "Reference" "#PWR0305"
+		(property "Reference" "#PWR0406"
 			(at 142.24 105.41 0)
 			(effects
@@
 			(project "Drone_Flight_Controller"
 				(path "/05daaa24-e506-4b9a-9564-8bf799413ca8/be1bc5c9-9814-4f01-a307-b935c6145e5a"
-					(reference "#PWR0305")
+					(reference "#PWR0406")
 					(unit 1)
 				)
@@
 		(dnp no)
 		(fields_autoplaced yes)
-		(property "Reference" "#PWR0308"
+		(property "Reference" "#PWR0408"
 			(at 195.58 152.4 0)
 			(effects
@@
 			(project "Drone_Flight_Controller"
 				(path "/05daaa24-e506-4b9a-9564-8bf799413ca8/be1bc5c9-9814-4f01-a307-b935c6145e5a"
-					(reference "#PWR0308")
+					(reference "#PWR0408")
 					(unit 1)
 				)
@@
 		(dnp no)
 		(fields_autoplaced yes)
-		(property "Reference" "#PWR0303"
+		(property "Reference" "#PWR0405"
 			(at 142.24 73.66 0)
 			(effects
@@
 			(project "Drone_Flight_Controller"
 				(path "/05daaa24-e506-4b9a-9564-8bf799413ca8/be1bc5c9-9814-4f01-a307-b935c6145e5a"
-					(reference "#PWR0303")
+					(reference "#PWR0405")
 					(unit 1)
 				)
@@
 		(on_board yes)
 		(dnp no)
-		(property "Reference" "C301"
+		(property "Reference" "C403"
 			(at 149.86 81.28 90)
 			(effects
@@
 			)
 		)
-		(property "Value" "1µF"
+		(property "Value" "1µ"
 			(at 149.86 83.82 90)
 			(effects
@@
 			(project ""
 				(path "/05daaa24-e506-4b9a-9564-8bf799413ca8/be1bc5c9-9814-4f01-a307-b935c6145e5a"
-					(reference "C301")
+					(reference "C403")
 					(unit 1)
 				)
@@
 		(on_board yes)
 		(dnp no)
-		(property "Reference" "U302"
+		(property "Reference" "U402"
 			(at 102.362 69.85 0)
 			(effects
@@
 			(project "Drone_Flight_Controller"
 				(path "/05daaa24-e506-4b9a-9564-8bf799413ca8/be1bc5c9-9814-4f01-a307-b935c6145e5a"
-					(reference "U302")
+					(reference "U402")
 					(unit 1)
 				)
@@
 		(on_board yes)
 		(dnp no)
-		(property "Reference" "SW301"
+		(property "Reference" "SW401"
 			(at 149.86 90.424 0)
 			(effects
@@
 			(project ""
 				(path "/05daaa24-e506-4b9a-9564-8bf799413ca8/be1bc5c9-9814-4f01-a307-b935c6145e5a"
-					(reference "SW301")
+					(reference "SW401")
 					(unit 1)
 				)
@@
 		(dnp no)
 		(fields_autoplaced yes)
-		(property "Reference" "C302"
+		(property "Reference" "C402"
 			(at 129.54 86.3599 0)
 			(effects
@@
 			)
 		)
-		(property "Value" "120nF"
+		(property "Value" "120n"
 			(at 129.54 88.8999 0)
 			(effects
@@
 			(project "Drone_Flight_Controller"
 				(path "/05daaa24-e506-4b9a-9564-8bf799413ca8/be1bc5c9-9814-4f01-a307-b935c6145e5a"
-					(reference "C302")
+					(reference "C402")
 					(unit 1)
 				)
@@
 		(dnp no)
 		(fields_autoplaced yes)
-		(property "Reference" "R301"
+		(property "Reference" "R401"
 			(at 88.9 62.23 90)
 			(effects
@@
 			(project ""
 				(path "/05daaa24-e506-4b9a-9564-8bf799413ca8/be1bc5c9-9814-4f01-a307-b935c6145e5a"
-					(reference "R301")
+					(reference "R401")
 					(unit 1)
 				)
@@
 		(on_board yes)
 		(dnp no)
-		(property "Reference" "C303"
+		(property "Reference" "C404"
 			(at 149.86 100.076 90)
 			(effects
@@
 			(project "Drone_Flight_Controller"
 				(path "/05daaa24-e506-4b9a-9564-8bf799413ca8/be1bc5c9-9814-4f01-a307-b935c6145e5a"
-					(reference "C303")
+					(reference "C404")
 					(unit 1)
 				)
@@
 		(on_board yes)
 		(dnp no)
-		(property "Reference" "R302"
+		(property "Reference" "R403"
 			(at 209.55 71.12 90)
 			(effects
@@
 			(project "Drone_Flight_Controller"
 				(path "/05daaa24-e506-4b9a-9564-8bf799413ca8/be1bc5c9-9814-4f01-a307-b935c6145e5a"
-					(reference "R302")
+					(reference "R403")
 					(unit 1)
 				)
@@
 		(dnp no)
 		(fields_autoplaced yes)
-		(property "Reference" "#PWR0301"
+		(property "Reference" "#PWR0407"
 			(at 195.58 67.31 0)
 			(effects
@@
 			(project "Drone_Flight_Controller"
 				(path "/05daaa24-e506-4b9a-9564-8bf799413ca8/be1bc5c9-9814-4f01-a307-b935c6145e5a"
-					(reference "#PWR0301")
+					(reference "#PWR0407")
 					(unit 1)
 				)
@@
 		(on_board yes)
 		(dnp no)
-		(property "Reference" "U301"
+		(property "Reference" "U401"
 			(at 52.07 86.36 0)
 			(effects
@@
 			(project "Drone_Flight_Controller"
 				(path "/05daaa24-e506-4b9a-9564-8bf799413ca8/be1bc5c9-9814-4f01-a307-b935c6145e5a"
-					(reference "U301")
+					(reference "U401")
 					(unit 1)
 				)
@@
 		(dnp no)
 		(fields_autoplaced yes)
-		(property "Reference" "R303"
+		(property "Reference" "R402"
 			(at 149.86 66.04 90)
 			(effects
@@
 			(project ""
 				(path "/05daaa24-e506-4b9a-9564-8bf799413ca8/be1bc5c9-9814-4f01-a307-b935c6145e5a"
-					(reference "R303")
+					(reference "R402")
 					(unit 1)
 				)
@@
 		(dnp no)
 		(fields_autoplaced yes)
-		(property "Reference" "#PWR0304"
+		(property "Reference" "#PWR0402"
 			(at 45.72 87.63 0)
 			(effects
@@
 			(project "Drone_Flight_Controller"
 				(path "/05daaa24-e506-4b9a-9564-8bf799413ca8/be1bc5c9-9814-4f01-a307-b935c6145e5a"
-					(reference "#PWR0304")
+					(reference "#PWR0402")
 					(unit 1)
 				)
@@
 		(on_board yes)
 		(dnp no)
-		(property "Reference" "C304"
+		(property "Reference" "C401"
 			(at 119.38 98.298 90)
 			(effects
@@
 			(project "Drone_Flight_Controller"
 				(path "/05daaa24-e506-4b9a-9564-8bf799413ca8/be1bc5c9-9814-4f01-a307-b935c6145e5a"
-					(reference "C304")
+					(reference "C401")
 					(unit 1)
 				)
@@
 		(dnp no)
 		(fields_autoplaced yes)
-		(property "Reference" "#PWR0306"
+		(property "Reference" "#PWR0401"
 			(at 43.18 115.57 0)
 			(effects
@@
 			(project "Drone_Flight_Controller"
 				(path "/05daaa24-e506-4b9a-9564-8bf799413ca8/be1bc5c9-9814-4f01-a307-b935c6145e5a"
-					(reference "#PWR0306")
-					(unit 1)
-				)
+					(reference "#PWR0401")
+					(unit 1)
+				)
