File: KiCAD/Drone_Flight_Controller/Peripherals.kicad_sch (KiCad schematic)
At the start: 57 parts, among them J1 XT60, J2 0.5mΩ high side shunt, Q1 2N2222A, U1 74AHC1G125, U2 74AHC1G125, U3 74AHC1G125, U4 74AHC1G125, U9 INA195

Commit message: routing
routing
Parts:
- added +5V2: +5V, TestPoint:TestPoint_Pad_D1.0mm, symbol Connector:TestPoint
- added 3V1: 3V3, TestPoint:TestPoint_Pad_D1.0mm, symbol Connector:TestPoint
- added C15: 10uF, Capacitor_SMD:C_0805_2012Metric, symbol Device:C_Small
- added C16: 100nF, Capacitor_SMD:C_0805_2012Metric, symbol Device:C_Small
- added GND2: GND, TestPoint:TestPoint_Pad_D1.0mm, symbol Connector:TestPoint
Connections:
- net +3V3: now also 3V1.1
- net +5V: now also +5V2.1, C15.1, C16.1
- net GND: now also C15.2, C16.2, GND2.1
